File: pcb/keys/client.kicad_pcb (KiCad board)
At the start: 2 copper layers, 80 x 40 mm, 16 parts, among them J1 Conn_01x04_Male, SW1 SW_Set, SW2 SW_Plus, SW3 SW_Minus, U1 TM1637, U2 CA56-12SEKWA

Commit message: Новая разводка
Parts:
- moved C2 25.4 mm to (101.3, 38.0), turned to 90 degrees
- moved C3 21.1 mm to (100.7, 66.0), turned to 0 degrees
- moved R2 17.2 mm to (105.3, 37.8), turned to 270 degrees
- moved R1 13.7 mm to (113.2, 37.7), turned to 270 degrees
- moved C1 9.39 mm to (109.7, 37.6), turned to 90 degrees
- moved C4 9.32 mm to (100.5, 62.2)
- moved SW1 5.08 mm to (160.0, 38.1), turned to 270 degrees
- moved SW2 5.08 mm to (160.0, 49.5), turned to 270 degrees
- moved SW3 5.08 mm to (160.0, 61.0), turned to 270 degrees
- moved J1 3.70 mm to (102.2, 52.7), turned to 270 degrees
- moved U2 1.53 mm to (115.4, 60.7)
- moved U1 0.64 mm to (140.5, 52.5), turned to 180 degrees
Routing:
- net GNDREF: track 76.0 -> 112.8 mm
- net VCC: track 56.9 -> 74.7 mm, vias 2 -> 0
- net Net-(C1-Pad2): track 78.7 -> 62.5 mm
- net Net-(U1-Pad6): track 42.7 -> 26.9 mm
- net Net-(SW1-Pad1): track 61.3 -> 46.8 mm, vias 1 -> 0
- net Net-(SW1-Pad2): track 60.0 -> 48.0 mm, vias 1 -> 0
- net Net-(U1-Pad9): track 29.6 -> 18.7 mm, vias 0 -> 1
- net Net-(U1-Pad13): track 25.2 -> 14.3 mm
- net Net-(U1-Pad8): track 24.6 -> 13.9 mm, vias 0 -> 1
- net Net-(SW2-Pad2): track 38.4 -> 49.1 mm
- net Net-(U1-Pad12): track 10.5 -> 18.9 mm, vias 0 -> 1
- net Net-(U1-Pad7): track 30.8 -> 23.6 mm, vias 1 -> 0
- net Net-(U1-Pad5): track 32.3 -> 25.4 mm, vias 1 -> 0
- net Net-(U1-Pad15): track 25.3 -> 27.9 mm, vias 1 -> 0
- net Net-(SW3-Pad2): track 63.4 -> 64.3 mm
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Other:
- net class Default: trace_width 0.25 -> 0.3
