File: pcb/motherboard/motherboard/motherboard.sch (KiCad schematic (older format))
At the start: 5 parts, among them J1 Power_Conn_01x02, J2 Sensor_Conn_01x03, J3 Display_01x04, U1 RobotDyn_NodeMCU

Commit message: Тесты дисплея
Parts:
- removed J2: Sensor_Conn_01x03, symbol Connector_Generic:Conn_01x03
- added J3, J4, J5, J6, J7, J8: Sensor_Conn_01x03, Connector_JST:JST_PH_B3B-PH-K_1x03_P2.00mm_Vertical, symbol Connector_Generic:Conn_01x03
- added R2, R3, R4, R5, R6: 47k, Resistor_SMD:R_1206_3216Metric_Pad1.42x1.75mm_HandSolder, symbol Device:R
- J1: renamed from J3; footprint (none) -> Connector_JST:JST_PH_B4B-PH-K_1x04_P2.00mm_Vertical
- J2: renamed from J1; footprint (none) -> Connector_JST:JST_PH_B2B-PH-K_1x02_P2.00mm_Vertical
- R1: footprint (none) -> Resistor_SMD:R_1206_3216Metric_Pad1.42x1.75mm_HandSolder
- U1: footprint (none) -> ESP8266:RobotDyn_NodeMCU
Connections:
- net labels added: 3.3V, GND, GPIO0, GPIO14, GPIO16, GPIO2, GPIO4, GPIO5
- net labels removed: диспллей_питаеться_от_5_надо_преобразователь_уровней
- wire segments 28 -> 96
- no-connect marks 11 -> 16
