File: pcb/motherboard/motherboard/motherboard.kicad_pcb (KiCad board)
At the start: 2 copper layers, 1 part, among them U1 RobotDyn_NodeMCU

Commit message: Тесты дисплея
Parts:
- added J1: Display_01x04, Connector_JST:JST_PH_B4B-PH-K_1x04_P2.00mm_Vertical, F.Cu at (112.8, 92.9)
- added J2: Power_Conn_01x02, Connector_JST:JST_PH_B2B-PH-K_1x02_P2.00mm_Vertical, F.Cu at (110.2, 126.9)
- added J3: Sensor_Conn_01x03, Connector_JST:JST_PH_B3B-PH-K_1x03_P2.00mm_Vertical, F.Cu at (167.6, 88.8)
- added J4: Sensor_Conn_01x03, Connector_JST:JST_PH_B3B-PH-K_1x03_P2.00mm_Vertical, F.Cu at (167.6, 97.4)
- added J5: Sensor_Conn_01x03, Connector_JST:JST_PH_B3B-PH-K_1x03_P2.00mm_Vertical, F.Cu at (167.6, 106.1)
- added J6: Sensor_Conn_01x03, Connector_JST:JST_PH_B3B-PH-K_1x03_P2.00mm_Vertical, F.Cu at (167.6, 115.7)
- added J7: Sensor_Conn_01x03, Connector_JST:JST_PH_B3B-PH-K_1x03_P2.00mm_Vertical, F.Cu at (167.6, 125.9)
- added J8: Sensor_Conn_01x03, Connector_JST:JST_PH_B3B-PH-K_1x03_P2.00mm_Vertical, F.Cu at (167.6, 135.8)
- added R1: 47k, Resistor_SMD:R_1206_3216Metric_Pad1.42x1.75mm_HandSolder, B.Cu at (164.1, 93.6)
- added R2: 47k, Resistor_SMD:R_1206_3216Metric_Pad1.42x1.75mm_HandSolder, B.Cu at (163.6, 98.9)
- added R3: 47k, Resistor_SMD:R_1206_3216Metric_Pad1.42x1.75mm_HandSolder, B.Cu at (163.6, 107.6)
- added R4: 47k, Resistor_SMD:R_1206_3216Metric_Pad1.42x1.75mm_HandSolder, B.Cu at (163.7, 117.2)
- added R5: 47k, Resistor_SMD:R_1206_3216Metric_Pad1.42x1.75mm_HandSolder, B.Cu at (166.2, 130.8)
- added R6: 47k, Resistor_SMD:R_1206_3216Metric_Pad1.42x1.75mm_HandSolder, B.Cu at (163.6, 138.3)
- added REF**: MountingHole_2.2mm_M2_DIN965_Pad, MountingHole:MountingHole_2.2mm_M2_DIN965_Pad, F.Cu at (181.8, 87.5)
- added REF**: MountingHole_2.2mm_M2_DIN965_Pad, MountingHole:MountingHole_2.2mm_M2_DIN965_Pad, F.Cu at (98.8, 87.5)
- added REF**: MountingHole_2.2mm_M2_DIN965_Pad, MountingHole:MountingHole_2.2mm_M2_DIN965_Pad, F.Cu at (98.8, 140.5)
- added REF**: MountingHole_2.2mm_M2_DIN965_Pad, MountingHole:MountingHole_2.2mm_M2_DIN965_Pad, F.Cu at (181.8, 140.5)
- moved U1 30.5 mm to (138.8, 111.5)
Connections:
- U1 pad 10: Net-(U1-Pad10) -> GND
- U1 pad 14: Net-(U1-Pad14) -> GND
- U1 pad 16: Net-(U1-Pad16) -> 3.3V
- U1 pad 17: Net-(U1-Pad17) -> GND
- U1 pad 23: Net-(U1-Pad23) -> GPIO14
- U1 pad 24: Net-(U1-Pad24) -> GND
- U1 pad 26: Net-(U1-Pad26) -> GPIO2
- U1 pad 27: Net-(U1-Pad27) -> GPIO0
- U1 pad 28: Net-(U1-Pad28) -> GPIO4
- U1 pad 29: Net-(U1-Pad29) -> GPIO5
- U1 pad 30: Net-(U1-Pad30) -> GPIO16
Routing:
- net GND: track 0.00 -> 206.5 mm
- net 3.3V: track 0.00 -> 102.1 mm
- net Net-(J1-Pad3): track 0.00 -> 52.7 mm
- net GPIO2: track 0.00 -> 39.3 mm
- net GPIO14: track 0.00 -> 36.0 mm
- net GPIO0: track 0.00 -> 27.7 mm
- net Net-(J1-Pad2): track 0.00 -> 24.1 mm
- net GPIO4: track 0.00 -> 20.9 mm
- net GPIO16: track 0.00 -> 20.1 mm
- net Net-(J1-Pad1): track 0.00 -> 20.0 mm
- net GPIO5: track 0.00 -> 17.8 mm
- added copper zone on B.Cu, net GND
Other:
- board outline added: 90 x 60 mm
- net class +5 added: clearance 0.8, trace_width 1, via_dia 0.8, via_drill 0.4
- net class Default: clearance 0.2 -> 0.7; trace_width 0.25 -> 0.9
- rule trace_clearance: 0.2 -> 0.7
- rule trace_min: 0.2 -> 0.4
- board text added: "Climate Control v1.1"
